File: kicad_Poolcontroller/kicad_Poolcontroller.sch (KiCad schematic (older format))
At the start: 34 parts, among them K1 SANYOU_SRD_Form_C, Q1 2N2219, Q2 2N2219, Q3 2N2219, Q4 2N2219, Q5 2N2219, Q6 2N2219, Q7 2N2219, Q8 2N2219

Commit message: .
Parts:
- added J1: Conn_02x02_Odd_Even, Connector_PinHeader_2.54mm:PinHeader_2x02_P2.54mm_Vertical, symbol Connector_Generic:Conn_02x02_Odd_Even
- added U3: L7809, symbol Regulator_Linear:L7809
- added U4: L7805, symbol Regulator_Linear:L7805
- added U5: LM317, symbol Regulator_Linear:LM317_3PinPackage
- U1: renamed from U?; symbol MCU_Microchip_ATtiny:ATtiny85V-10PU -> Pool_Controller-rescue:ATtiny85V-10PU-MCU_Microchip_ATtiny
- gave numbers to parts that had none: 1
Changed lines of the file:
@@
 EESchema Schematic File Version 4
+LIBS:Pool_Controller-cache
 EELAYER 30 0
 EELAYER END
@@
 $EndDescr
 $Comp
-L 74xx:74HC595 U?
+L 74xx:74HC595 U2
 U 1 1 601F13DC
 P 4550 1400
-F 0 "U?" H 4550 2181 50  0000 C CNN
-F 1 "74HC595" H 4550 2090 50  0000 C CNN
+F 0 "U2" H 4550 2181 50  0000 C CNN
+F 1 "74HC595" H 4550 2090 50  0001 C CNN
 F 2 "" H 4550 1400 50  0001 C CNN
 F 3 "http://www.ti.com/lit/ds/symlink/sn74hc595.pdf" H 4550 1400 50  0001 C CNN
@@
 $EndComp
 $Comp
-L MCU_Microchip_ATtiny:ATtiny85V-10PU U?
+L Pool_Controller-rescue:ATtiny85V-10PU-MCU_Microchip_ATtiny U1
 U 1 1 601F2825
 P 2850 1400
-F 0 "U?" H 2320 1446 50  0000 R CNN
-F 1 "ATtiny85V-10PU" H 2320 1355 50  0000 R CNN
+F 0 "U1" H 2320 1446 50  0000 R CNN
+F 1 "ATtiny85V-10PU" H 2320 1355 50  0001 R CNN
 F 2 "Package_DIP:DIP-8_W7.62mm" H 2850 1400 50  0001 C CIN
 F 3 "http://ww1.microchip.com/downloads/en/DeviceDoc/atmel-2586-avr-8-bit-microcontroller-attiny25-attiny45-attiny85_datasheet.pdf" H 2850 1400 50  0001 C CNN
@@
 Wire Wire Line
 	5800 4600 4450 4600
+$Comp
+L Regulator_Linear:L7805 U4
+U 1 1 60538E17
+P 9100 4250
+F 0 "U4" H 9100 4492 50  0000 C CNN
+F 1 "L7805" H 9100 4401 50  0000 C CNN
+F 2 "" H 9125 4100 50  0001 L CIN
+F 3 "http://www.st.com/content/ccc/resource/technical/document/datasheet/41/4f/b3/b0/12/d4/47/88/CD00000444.pdf/files/CD00000444.pdf/jcr:content/translations/en.CD00000444.pdf" H 9100 4200 50  0001 C CNN
+	1    9100 4250
+	1    0    0    -1
+$EndComp
+$Comp
+L Regulator_Linear:L7809 U3
+U 1 1 60539486
+P 8100 4250
+F 0 "U3" H 8100 4492 50  0000 C CNN
+F 1 "L7809" H 8100 4401 50  0000 C CNN
+F 2 "" H 8125 4100 50  0001 L CIN
+F 3 "http://www.st.com/content/ccc/resource/technical/document/datasheet/41/4f/b3/b0/12/d4/47/88/CD00000444.pdf/files/CD00000444.pdf/jcr:content/translations/en.CD00000444.pdf" H 8100 4200 50  0001 C CNN
+	1    8100 4250
+	1    0    0    -1
+$EndComp
+$Comp
+L Regulator_Linear:LM317_3PinPackage U5
+U 1 1 60539C18
+P 10000 4250
+F 0 "U5" H 10000 4492 50  0000 C CNN
+F 1 "LM317" H 10000 4401 50  0000 C CNN
+F 2 "" H 10000 4500 50  0001 C CIN
+F 3 "http://www.ti.com/lit/ds/symlink/lm317.pdf" H 10000 4250 50  0001 C CNN
+	1    10000 4250
+	1    0    0    -1
+$EndComp
+$Comp
+L Connector_Generic:Conn_02x02_Odd_Even J1
+U 1 1 60581858
+P 7350 4250
+F 0 "J1" H 7400 4375 50  0000 C CNN
+F 1 "Conn_02x02_Odd_Even" H 7400 4376 50  0001 C CNN
+F 2 "Connector_PinHeader_2.54mm:PinHeader_2x02_P2.54mm_Vertical" H 7400 4376 50  0001 C CNN
+F 3 "~" H 7350 4250 50  0001 C CNN
+	1    7350 4250
+	1    0    0    -1
+$EndComp
 $EndSCHEMATC

Commit message: .
Parts:
- added C1, C3: 220u, symbol pspice:C
- added C2, C4: 47u, symbol pspice:C
- added J1: Conn_02x01, symbol Connector_Generic:Conn_02x01
- added R? (x2): R, symbol Device:R
- U1: symbol Pool_Controller-rescue:ATtiny85V-10PU-MCU_Microchip_ATtiny -> kicad_Poolcontroller-rescue:ATtiny85V-10PU-MCU_Microchip_ATtiny-Pool_Controller-rescue
- renumbered J1 to J2
Connections:
- net labels added: 3.3V, 5V
- wire segments 158 -> 193
Other:
- moved on the sheet: J2, U3, U4, U5
Changed lines of the file:
@@
 EESchema Schematic File Version 4
-LIBS:Pool_Controller-cache
 EELAYER 30 0
 EELAYER END
@@
 $EndComp
 $Comp
-L Pool_Controller-rescue:ATtiny85V-10PU-MCU_Microchip_ATtiny U1
+L kicad_Poolcontroller-rescue:ATtiny85V-10PU-MCU_Microchip_ATtiny-Pool_Controller-rescue U1
 U 1 1 601F2825
 P 2850 1400
@@
 L Regulator_Linear:L7805 U4
 U 1 1 60538E17
-P 9100 4250
-F 0 "U4" H 9100 4492 50  0000 C CNN
-F 1 "L7805" H 9100 4401 50  0000 C CNN
-F 2 "" H 9125 4100 50  0001 L CIN
-F 3 "http://www.st.com/content/ccc/resource/technical/document/datasheet/41/4f/b3/b0/12/d4/47/88/CD00000444.pdf/files/CD00000444.pdf/jcr:content/translations/en.CD00000444.pdf" H 9100 4200 50  0001 C CNN
-	1    9100 4250
+P 9300 4250
+F 0 "U4" H 9300 4492 50  0000 C CNN
+F 1 "L7805" H 9300 4401 50  0000 C CNN
+F 2 "" H 9325 4100 50  0001 L CIN
+F 3 "http://www.st.com/content/ccc/resource/technical/document/datasheet/41/4f/b3/b0/12/d4/47/88/CD00000444.pdf/files/CD00000444.pdf/jcr:content/translations/en.CD00000444.pdf" H 9300 4200 50  0001 C CNN
+	1    9300 4250
+	1    0    0    -1
+$EndComp
+$Comp
+L Regulator_Linear:LM317_3PinPackage U5
+U 1 1 60539C18
+P 10250 4250
+F 0 "U5" H 10250 4492 50  0000 C CNN
+F 1 "LM317" H 10250 4401 50  0000 C CNN
+F 2 "" H 10250 4500 50  0001 C CIN
+F 3 "http://www.ti.com/lit/ds/symlink/lm317.pdf" H 10250 4250 50  0001 C CNN
+	1    10250 4250
+	1    0    0    -1
+$EndComp
+$Comp
+L Connector_Generic:Conn_02x02_Odd_Even J2
+U 1 1 60581858
+P 6900 4250
+F 0 "J2" H 6950 4375 50  0000 C CNN
+F 1 "Conn_02x02_Odd_Even" H 6950 4376 50  0001 C CNN
+F 2 "Connector_PinHeader_2.54mm:PinHeader_2x02_P2.54mm_Vertical" H 6950 4376 50  0001 C CNN
+F 3 "~" H 6900 4250 50  0001 C CNN
+	1    6900 4250
 	1    0    0    -1
 $EndComp
@@
 L Regulator_Linear:L7809 U3
 U 1 1 60539486
-P 8100 4250
-F 0 "U3" H 8100 4492 50  0000 C CNN
-F 1 "L7809" H 8100 4401 50  0000 C CNN
-F 2 "" H 8125 4100 50  0001 L CIN
-F 3 "http://www.st.com/content/ccc/resource/technical/document/datasheet/41/4f/b3/b0/12/d4/47/88/CD00000444.pdf/files/CD00000444.pdf/jcr:content/translations/en.CD00000444.pdf" H 8100 4200 50  0001 C CNN
-	1    8100 4250
-	1    0    0    -1
-$EndComp
-$Comp
-L Regulator_Linear:LM317_3PinPackage U5
-U 1 1 60539C18
-P 10000 4250
-F 0 "U5" H 10000 4492 50  0000 C CNN
-F 1 "LM317" H 10000 4401 50  0000 C CNN
-F 2 "" H 10000 4500 50  0001 C CIN
-F 3 "http://www.ti.com/lit/ds/symlink/lm317.pdf" H 10000 4250 50  0001 C CNN
-	1    10000 4250
-	1    0    0    -1
-$EndComp
-$Comp
-L Connector_Generic:Conn_02x02_Odd_Even J1
-U 1 1 60581858
-P 7350 4250
-F 0 "J1" H 7400 4375 50  0000 C CNN
-F 1 "Conn_02x02_Odd_Even" H 7400 4376 50  0001 C CNN
-F 2 "Connector_PinHeader_2.54mm:PinHeader_2x02_P2.54mm_Vertical" H 7400 4376 50  0001 C CNN
-F 3 "~" H 7350 4250 50  0001 C CNN
-	1    7350 4250
-	1    0    0    -1
-$EndComp
+P 8000 4250
+F 0 "U3" H 8000 4492 50  0000 C CNN
+F 1 "L7809" H 8000 4401 50  0000 C CNN
+F 2 "" H 8025 4100 50  0001 L CIN
+F 3 "http://www.st.com/content/ccc/resource/technical/document/datasheet/41/4f/b3/b0/12/d4/47/88/CD00000444.pdf/files/CD00000444.pdf/jcr:content/translations/en.CD00000444.pdf" H 8000 4200 50  0001 C CNN
+	1    8000 4250
+	1    0    0    -1
+$EndComp
+$Comp
+L pspice:C C2
+U 1 1 60613901
+P 8400 4800
+F 0 "C2" H 8578 4800 50  0000 L CNN
+F 1 "47u" H 8578 4755 50  0001 L CNN
+F 2 "" H 8400 4800 50  0001 C CNN
+F 3 "~" H 8400 4800 50  0001 C CNN
+	1    8400 4800
+	1    0    0    -1
+$EndComp
+$Comp
+L pspice:C C1
+U 1 1 60612DCD
+P 7600 4800
+F 0 "C1" H 7778 4800 50  0000 L CNN
+F 1 "220u" H 7778 4755 50  0001 L CNN
+F 2 "" H 7600 4800 50  0001 C CNN
+F 3 "~" H 7600 4800 50  0001 C CNN
+	1    7600 4800
+	1    0    0    -1
+$EndComp
+$Comp
+L pspice:C C3
+U 1 1 6061E85E
+P 8900 4800
+F 0 "C3" H 9078 4800 50  0000 L CNN
+F 1 "220u" H 9078 4755 50  0001 L CNN
+F 2 "" H 8900 4800 50  0001 C CNN
+F 3 "~" H 8900 4800 50  0001 C CNN
+	1    8900 4800
+	1    0    0    -1
+$EndComp
+$Comp
+L pspice:C C4
+U 1 1 6061FCB8
+P 9700 4800
+F 0 "C4" H 9878 4800 50  0000 L CNN
+F 1 "47u" H 9878 4755 50  0001 L CNN
+F 2 "" H 9700 4800 50  0001 C CNN
+F 3 "~" H 9700 4800 50  0001 C CNN
+	1    9700 4800
+	1    0    0    -1
+$EndComp
+Text HLabel 7300 4350 2    50   Output ~ 0
+5V
+$Comp
+L Connector_Generic:Conn_02x01 J1
+U 1 1 6063541F
+P 6900 5250
+F 0 "J1" H 6950 5375 50  0000 C CNN
+F 1 "Conn_02x01" H 6950 5376 50  0001 C CNN
+F 2 "" H 6900 5250 50  0001 C CNN
+F 3 "~" H 6900 5250 50  0001 C CNN
+	1    6900 5250
+	1    0    0    -1
+$EndComp
+Wire Wire Line
+	7200 5250 7600 5250
+Wire Wire Line
+	7600 5250 7600 5050
+Wire Wire Line
+	9700 5050 9700 5250
+Wire Wire Line
+	9700 5250 8900 5250
+Connection ~ 7600 5250
+Wire Wire Line
+	8400 5050 8400 5250
+Connection ~ 8400 5250
+Wire Wire Line
+	8400 5250 7600 5250
+Wire Wire Line
+	8900 5050 8900 5250
+Connection ~ 8900 5250
+Wire Wire Line
+	8900 5250 8400 5250
+Wire Wire Line
+	7600 4550 7600 4250
+Wire Wire Line
+	7600 4250 7700 4250
+Wire Wire Line
+	7600 4250 7200 4250
+Connection ~ 7600 4250
+Wire Wire Line
+	8300 4250 8400 4250
+Wire Wire Line
+	8400 4250 8400 4550
+Wire Wire Line
+	8400 4250 8650 4250
+Connection ~ 8400 4250
+Wire Wire Line
+	8900 4250 8900 4550
+Connection ~ 8900 4250
+Wire Wire Line
+	8900 4250 9000 4250
+Text HLabel 8650 4100 1    50   Input ~ 0
+5V
+Wire Wire Line
+	8650 4100 8650 4250
+Connection ~ 8650 4250
+Wire Wire Line
+	8650 4250 8900 4250
+Wire Wire Line
+	6700 5250 6650 5250
+Wire Wire Line
+	6650 5250 6650 4350
+Wire Wire Line
+	6650 4250 6700 4250
+Wire Wire Line
+	6650 4350 6700 4350
+Connection ~ 6650 4350
+Wire Wire Line
+	6650 4350 6650 4250
+Wire Wire Line
+	9600 4250 9700 4250
+Wire Wire Line
+	9700 4250 9700 4550
+Wire Wire Line
+	9700 4250 9950 4250
+Connection ~ 9700 4250
+$Comp
+L Device:R R?
+U 1 1 606B34ED
+P 10250 5050
+F 0 "R?" H 10320 5096 50  0000 L CNN
+F 1 "R" H 10320 5005 50  0000 L CNN
+F 2 "" V 10180 5050 50  0001 C CNN
+F 3 "~" H 10250 5050 50  0001 C CNN
+	1    10250 5050
+	1    0    0    -1
+$EndComp
+$Comp
+L Device:R R?
+U 1 1 606B3F3F
+P 10700 4500
+F 0 "R?" H 10630 4454 50  0000 R CNN
+F 1 "R" H 10630 4545 50  0000 R CNN
+F 2 "" V 10630 4500 50  0001 C CNN
+F 3 "~" H 10700 4500 50  0001 C CNN
+	1    10700 4500
+	-1   0    0    1
+$EndComp
+Wire Wire Line
+	10250 4550 10250 4750
+Wire Wire Line
+	10700 4650 10700 4750
+Wire Wire Line
+	10700 4750 10250 4750
+Connection ~ 10250 4750
+Wire Wire Line
+	10250 4750 10250 4900
+Wire Wire Line
+	9700 5250 10250 5250
+Wire Wire Line
+	10250 5250 10250 5200
+Connection ~ 9700 5250
+Wire Wire Line
+	10550 4250 10700 4250
+Wire Wire Line
+	10700 4250 10700 4350
+Text HLabel 10900 4250 2    50   Output ~ 0
+3.3V
+Wire Wire Line
+	10700 4250 10900 4250
+Connection ~ 10700 4250
 $EndSCHEMATC

Commit message: att
Parts:
- added J4 (x2): Conn_02x01, Connector_PinHeader_2.54mm:PinHeader_2x01_P2.54mm_Vertical, symbol Connector_Generic:Conn_02x01
- added J?: Conn_02x02_Odd_Even, Connector_PinHeader_2.54mm:PinHeader_2x02_P2.54mm_Vertical, symbol Connector_Generic:Conn_02x02_Odd_Even
- J1: footprint (none) -> Connector_PinHeader_2.54mm:PinHeader_2x01_P2.54mm_Vertical
- R1, R2, R3, R4, R5, R6, R7, R8: footprint (none) -> Resistor_THT:R_Axial_DIN0207_L6.3mm_D2.5mm_P10.16mm_Horizontal
- R1: renamed from R?; value R -> 220R
- R2: renamed from R?; value R -> 360R
- U1: footprint Package_DIP:DIP-8_W7.62mm -> Package_DIP:DIP-6_W7.62mm_Socket
- U2: footprint (none) -> Package_DIP:DIP-16_W7.62mm_Socket
- U3, U4, U5: footprint (none) -> Package_TO_SOT_THT:TO-220-3_Vertical
- gave numbers to parts that had none: 14
Connections:
- net +12V: now also J1.1 (Pin_1), J2.1 (Pin_1), J2.3 (Pin_3), J4.2 (Pin_2), J4.2 (Pin_2); no longer K1.1, K2.1, K3.1, K4.1, K5.1, K6.1, K7.1, K8.1
- net 5V: no longer C2.1, C3.1, U3.3 (OUT), U4.1 (IN)
- net GND: now also C1.2, C2.2, C3.2, C4.2, J1.2 (Pin_2), R1.2, U1.4 (GND), U2.8 (GND), U3.2 (GND), U4.2 (GND)
- net K1: no longer D2.1 (K), D3.1 (K), D4.1 (K), D5.1 (K), D6.1 (K), D7.1 (K), D8.1 (K), K2.5, K3.5, K4.5, K5.5, K6.5, K7.5, K8.5
- net K2: now also D2.1 (K), K2.5
- net K3: now also D3.1 (K), K3.5
- net K4: now also D4.1 (K), K4.5
- net K5: now also D5.1 (K), K5.5
- net K6: now also D6.1 (K), K6.5
- net K7: now also D7.1 (K), K7.5
- net K8: now also D8.1 (K), K8.5
- net at U2.10 (~SRCLR): now also U1.6 (PB1)
- net at U2.11 (SRCLK): now also U1.5 (AREF/PB0)
- net at U2.12 (RCLK): now also U1.7 (PB2)
- net +5V: now reaches U2.16 (VCC)
- net +5V: now also C4.1, U1.8 (VCC), U4.3 (OUT), U5.3 (VI)
- net at U1.2 (XTAL1/PB3): now also J?.4 (Pin_4)
- net at U1.3 (XTAL2/PB4): now also J?.2 (Pin_2)
- net 3.3V renamed +3.3V
- new net: J4.1 (Pin_1), K1.1, K2.1, K3.1, K4.1
- new net: J4.1 (Pin_1), K5.1, K6.1, K7.1, K8.1
- new net: C2.1, C3.1, U3.3 (OUT), U4.1 (IN)
Other:
- moved on the sheet: D1, D2, D3, D4, D5, D6, D7, D8, K1, K2, K3, K4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

Commit message: att
Parts:
- removed J4: Conn_02x01, Connector_PinHeader_2.54mm:PinHeader_2x01_P2.54mm_Vertical, symbol Connector_Generic:Conn_02x01
- C1, C2, C3, C4: footprint (none) -> Capacitor_THT:CP_Radial_D8.0mm_P3.50mm
- Q1, Q2, Q3, Q4, Q5, Q6, Q7, Q8: footprint Package_TO_SOT_THT:TO-39-3 -> Package_TO_SOT_THT:TO-92
- R10: renamed from R2; footprint (none) -> Resistor_THT:R_Axial_DIN0207_L6.3mm_D2.5mm_P10.16mm_Horizontal
- R9: renamed from R1; footprint (none) -> Resistor_THT:R_Axial_DIN0207_L6.3mm_D2.5mm_P10.16mm_Horizontal
- gave numbers to parts that had none: 1
Connections:
- net +12V: now also U2.10 (~SRCLR)
- net +5V: no longer C4.1, U4.3 (OUT), U5.3 (VI)
- net GND: now also U2.13 (~OE)
- net at U1.6 (PB1): now also U2.14 (SER); no longer U2.10 (~SRCLR)
- net at J4.1 (Pin_1), K1.1, K2.1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: now also K5.1, K6.1, K7.1, K8.1
- new net: C4.1, U4.3 (OUT), U5.3 (VI)
Other:
- moved on the sheet: C1, C2, C3, C4, D5, D6, D7, D8, J1, J2, J4, K5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

Commit message: att
Parts:
- removed J4: Conn_02x01, Connector_PinHeader_2.54mm:PinHeader_2x01_P2.54mm_Vertical, symbol Connector_Generic:Conn_02x01
- added J10, J11, J12, J13, J7, J8, J9: Conn_02x01, TerminalBlock:TerminalBlock_bornier-2_P5.08mm, symbol Connector_Generic:Conn_02x01
- added J4: Conn_01x04, Connector_PinSocket_2.54mm:PinSocket_1x04_P2.54mm_Vertical, symbol Connector_Generic:Conn_01x04
- added J5: ESP01, Connector_PinSocket_2.54mm:PinSocket_2x04_P2.54mm_Vertical, symbol Connector_Generic:Conn_02x04_Odd_Even
- added J6: Conn_01x03, TerminalBlock:TerminalBlock_bornier-3_P5.08mm, symbol Connector_Generic:Conn_01x03
- C1, C2, C3, C4: footprint Capacitor_THT:CP_Radial_D8.0mm_P3.50mm -> Capacitor_THT:CP_Radial_D5.0mm_P2.50mm
- U1: footprint Package_DIP:DIP-6_W7.62mm_Socket -> Package_DIP:DIP-8_W7.62mm_Socket
- U5: footprint Package_TO_SOT_THT:TO-220-3_Vertical -> Package_TO_SOT_THT:TO-220-3_Horizontal_TabDown
Connections:
- net +12V: now also J3.2 (Pin_2); no longer Q1.3 (C), Q2.3 (C), Q3.3 (C), Q4.3 (C), Q5.3 (C), Q6.3 (C), Q7.3 (C), Q8.3 (C)
- net +3.3V: now also J4.1 (Pin_1), J5.8 (Pin_8)
- net +5V: no longer U1.8 (VCC)
- net GND: now also J3.3 (Pin_3), J4.4 (Pin_4), J5.1 (Pin_1)
- net EN: now reaches U1.1 (~RESET~/PB5)
- net EN: now also J5.4 (Pin_4)
- net at J3.4 (Pin_4): no longer U1.2 (XTAL1/PB3)
- net TX: now reaches U1.3 (XTAL2/PB4)
- net TX: now also J4.2 (Pin_2), J5.2 (Pin_2); no longer J3.2 (Pin_2)
- net at K1.3: now also J9.2 (Pin_2)
- net at K1.4: now also J9.1 (Pin_1)
- net at K2.3: now also J8.2 (Pin_2)
- net at K2.4: now also J8.1 (Pin_1)
- net at K3.3: now also J7.2 (Pin_2)
- net at K3.4: now also J7.1 (Pin_1)
- net at K4.3: now also J6.3 (Pin_3)
- net at K4.4: now also J6.1 (Pin_1)
- net at K5.3: now also J10.2 (Pin_2)
- net at K5.4: now also J10.1 (Pin_1)
- net at K6.3: now also J11.2 (Pin_2)
- net at K6.4: now also J11.1 (Pin_1)
- net at K7.3: now also J12.2 (Pin_2)
- net at K7.4: now also J12.1 (Pin_1)
- net at K8.3: now also J13.2 (Pin_2)
- net at K8.4: now also J13.1 (Pin_1)
- net at J3.1 (Pin_1): now also Q1.3 (C), Q2.3 (C), Q3.3 (C), Q4.3 (C), Q5.3 (C), Q6.3 (C), Q7.3 (C), Q8.3 (C)
- new net: J6.2 (Pin_2), K4.1
- new net RX: J4.3 (Pin_3), J5.7 (Pin_7), U1.2 (XTAL1/PB3)
- now unconnected: K1.1, K2.1, K3.1, K5.1, K6.1, K7.1, K8.1
Other:
- moved on the sheet: Q1, Q2, Q3, Q4, Q5, Q6, Q7, Q8, U1

Commit message: att
Parts:
- removed J10, J11, J12, J13, J7, J8, J9: Conn_02x01, TerminalBlock:TerminalBlock_bornier-2_P5.08mm, symbol Connector_Generic:Conn_02x01
- removed J6: Conn_01x03, TerminalBlock:TerminalBlock_bornier-3_P5.08mm, symbol Connector_Generic:Conn_01x03
- added J10, J11, J12, J13, J6, J7, J8, J9: Conn_01x04, Connector_PinHeader_2.00mm:PinHeader_1x04_P2.00mm_Vertical, symbol Connector_Generic:Conn_01x04
Connections:
- net at K1.1: now also J9.4 (Pin_4)
- net at K1.3: now also J9.2 (Pin_2)
- net at K1.4: now also J9.1 (Pin_1)
- net at K2.1: now also J8.4 (Pin_4)
- net at K2.3: now also J8.2 (Pin_2)
- net at K2.4: now also J8.1 (Pin_1)
- net at K3.1: now also J7.4 (Pin_4)
- net at K3.3: now also J7.2 (Pin_2)
- net at K3.4: now also J7.1 (Pin_1)
- net at K4.1: now also J6.4 (Pin_4)
- net at K4.3: now also J6.2 (Pin_2)
- net at K4.4: now also J6.1 (Pin_1)
- net at K5.1: now also J10.4 (Pin_4)
- net at K5.3: now also J10.2 (Pin_2)
- net at K5.4: now also J10.1 (Pin_1)
- net at K6.1: now also J11.4 (Pin_4)
- net at K6.3: now also J11.2 (Pin_2)
- net at K6.4: now also J11.1 (Pin_1)
- net at K7.1: now also J12.4 (Pin_4)
- net at K7.3: now also J12.2 (Pin_2)
- net at K7.4: now also J12.1 (Pin_1)
- net at K8.1: now also J13.4 (Pin_4)
- net at K8.3: now also J13.2 (Pin_2)
- net at K8.4: now also J13.1 (Pin_1)
