File: kicad_Poolcontroller/kicad_Poolcontroller.sch (KiCad schematic (older format))
At the start: 56 parts, among them J1 Conn_02x01, J10 Conn_01x04, J11 Conn_01x04, J12 Conn_01x04, J13 Conn_01x04, J2 Conn_02x02_Odd_Even, J3 Conn_02x02_Odd_Even, J4 Conn_01x04, J5 ESP01, J6 Conn_01x04, J7 Conn_01x04, J8 Conn_01x04, J9 Conn_01x04, K1 SANYOU_SRD_Form_C, K2 SANYOU_SRD_Form_C, K3 SANYOU_SRD_Form_C, K4 SANYOU_SRD_Form_C, K5 SANYOU_SRD_Form_C, K6 SANYOU_SRD_Form_C, K7 SANYOU_SRD_Form_C, K8 SANYOU_SRD_Form_C, Q1 2N2219, Q2 2N2219, Q3 2N2219, Q4 2N2219, Q5 2N2219, Q6 2N2219, Q7 2N2219, Q8 2N2219, U1 ATtiny85V-10PU, U2 74HC595, U3 L7809, U4 L7805, U5 LM317

Commit message: att
Parts:
- J10, J11, J12, J13, J6, J7, J8, J9: footprint Connector_PinHeader_2.00mm:PinHeader_1x04_P2.00mm_Vertical -> TerminalBlock:TerminalBlock_bornier-4_P5.08mm
Connections:
- net +5V: now also J2.4 (Pin_4)
Changed lines of the file:
@@
 $EndComp
 Text HLabel 7350 4350 2    50   Output ~ 0
-5V
++5V
 $Comp
 L Connector_Generic:Conn_02x01 J1
@@
 Wire Wire Line
 	5500 4550 5500 4600
-Wire Wire Line
-	5500 4600 5850 4600
 $Comp
 L power:GND #PWR0101
@@
 F 0 "J6" V 5600 3650 50  0000 R CNN
 F 1 "Conn_01x04" V 5373 3362 50  0001 R CNN
-F 2 "Connector_PinHeader_2.00mm:PinHeader_1x04_P2.00mm_Vertical" H 5500 3650 50  0001 C CNN
+F 2 "TerminalBlock:TerminalBlock_bornier-4_P5.08mm" H 5500 3650 50  0001 C CNN
 F 3 "~" H 5500 3650 50  0001 C CNN
 	1    5500 3650
@@
 	1    0    0    -1
 $EndComp
+Wire Wire Line
+	5350 5350 5350 5450
+Wire Wire Line
+	5450 5350 5450 5400
+Wire Wire Line
+	5450 5400 5550 5400
+Wire Wire Line
+	5550 5400 5550 5450
+Wire Wire Line
+	5450 6050 5450 6200
+Wire Wire Line
+	5450 6200 5800 6200
+Wire Wire Line
+	5800 6200 5800 5450
+Wire Wire Line
+	5800 5450 5650 5450
+Wire Wire Line
+	5650 5450 5650 5350
+Wire Wire Line
+	5850 4600 5850 3950
+Wire Wire Line
+	5500 4600 5850 4600
+Wire Wire Line
+	5850 3950 5700 3950
+Wire Wire Line
+	4350 3850 4350 3950
+Wire Wire Line
+	4350 3950 4500 3950
+Wire Wire Line
+	4500 3950 4500 4600
+Wire Wire Line
+	4500 4600 4150 4600
+Wire Wire Line
+	4150 4600 4150 4550
+Wire Wire Line
+	4250 3950 4250 3900
+Wire Wire Line
+	4250 3900 4150 3900
+Wire Wire Line
+	4150 3900 4150 3850
+Wire Wire Line
+	4050 3850 4050 3950
+Wire Wire Line
+	3050 3850 3050 3950
+Wire Wire Line
+	3050 3950 3200 3950
+Wire Wire Line
+	3200 3950 3200 4600
+Wire Wire Line
+	3200 4600 2850 4600
+Wire Wire Line
+	2850 4600 2850 4550
+Wire Wire Line
+	2850 3850 2850 3900
+Wire Wire Line
+	2850 3900 2950 3900
+Wire Wire Line
+	2950 3900 2950 3950
+Wire Wire Line
+	2750 3850 2750 3950
+Wire Wire Line
+	1400 3850 1400 3950
+Wire Wire Line
+	1500 3850 1500 3900
+Wire Wire Line
+	1500 3900 1600 3900
+Wire Wire Line
+	1600 3900 1600 3950
+Wire Wire Line
+	1700 3850 1700 4000
+Wire Wire Line
+	1700 4000 1850 4000
+Wire Wire Line
+	1850 4000 1850 4600
+Wire Wire Line
+	1850 4600 1500 4600
+Wire Wire Line
+	1500 4600 1500 4550
+Wire Wire Line
+	1350 5350 1350 5450
+Wire Wire Line
+	1450 5350 1450 5400
+Wire Wire Line
+	1450 5400 1550 5400
+Wire Wire Line
+	1550 5400 1550 5450
+Wire Wire Line
+	1650 5350 1650 5500
+Wire Wire Line
+	1650 5500 1800 5500
+Wire Wire Line
+	1800 5500 1800 6100
+Wire Wire Line
+	1800 6100 1450 6100
+Wire Wire Line
+	1450 6100 1450 6050
+Wire Wire Line
+	2700 5350 2700 5450
+Wire Wire Line
+	2800 5350 2800 5400
+Wire Wire Line
+	2800 5400 2900 5400
+Wire Wire Line
+	2900 5400 2900 5450
+Wire Wire Line
+	3000 5350 3000 5500
+Wire Wire Line
+	3000 5500 3150 5500
+Wire Wire Line
+	3150 5500 3150 6100
+Wire Wire Line
+	3150 6100 2800 6100
+Wire Wire Line
+	2800 6100 2800 6050
+Wire Wire Line
+	4000 5350 4000 5450
+Wire Wire Line
+	4100 5350 4100 5400
+Wire Wire Line
+	4100 5400 4200 5400
+Wire Wire Line
+	4200 5400 4200 5450
+Wire Wire Line
+	4300 5350 4300 5500
+Wire Wire Line
+	4300 5500 4450 5500
+Wire Wire Line
+	4450 5500 4450 6100
+Wire Wire Line
+	4450 6100 4100 6100
+Wire Wire Line
+	4100 6100 4100 6050
+$Comp
+L Connector_Generic:Conn_01x04 J8
+U 1 1 60893E6F
+P 2850 3650
+F 0 "J8" V 2950 3650 50  0000 R CNN
+F 1 "Conn_01x04" V 2723 3362 50  0001 R CNN
+F 2 "TerminalBlock:TerminalBlock_bornier-4_P5.08mm" H 2850 3650 50  0001 C CNN
+F 3 "~" H 2850 3650 50  0001 C CNN
+	1    2850 3650
+	0    -1   -1   0
+$EndComp
+$Comp
+L Connector_Generic:Conn_01x04 J9
+U 1 1 6080408C
+P 1500 3650
+F 0 "J9" V 1600 3650 50  0000 R CNN
+F 1 "Conn_01x04" V 1373 3362 50  0001 R CNN
+F 2 "TerminalBlock:TerminalBlock_bornier-4_P5.08mm" H 1500 3650 50  0001 C CNN
+F 3 "~" H 1500 3650 50  0001 C CNN
+	1    1500 3650
+	0    -1   -1   0
+$EndComp
+$Comp
+L Connector_Generic:Conn_01x04 J13
+U 1 1 608075D9
+P 5450 5150
+F 0 "J13" V 5550 5150 50  0000 R CNN
+F 1 "Conn_01x04" V 5323 4862 50  0001 R CNN
+F 2 "TerminalBlock:TerminalBlock_bornier-4_P5.08mm" H 5450 5150 50  0001 C CNN
+F 3 "~" H 5450 5150 50  0001 C CNN
+	1    5450 5150
+	0    -1   -1   0
+$EndComp
+$Comp
+L Connector_Generic:Conn_01x04 J12
+U 1 1 60806A87
+P 4100 5150
+F 0 "J12" V 4200 5150 50  0000 R CNN
+F 1 "Conn_01x04" V 3973 4862 50  0001 R CNN
+F 2 "TerminalBlock:TerminalBlock_bornier-4_P5.08mm" H 4100 5150 50  0001 C CNN
+F 3 "~" H 4100 5150 50  0001 C CNN
+	1    4100 5150
+	0    -1   -1   0
+$EndComp
+$Comp
+L Connector_Generic:Conn_01x04 J11
+U 1 1 608060CB
+P 2800 5150
+F 0 "J11" V 2900 5150 50  0000 R CNN
+F 1 "Conn_01x04" V 2673 4862 50  0001 R CNN
+F 2 "TerminalBlock:TerminalBlock_bornier-4_P5.08mm" H 2800 5150 50  0001 C CNN
+F 3 "~" H 2800 5150 50  0001 C CNN
+	1    2800 5150
+	0    -1   -1   0
+$EndComp
+$Comp
+L Connector_Generic:Conn_01x04 J10
+U 1 1 60805349
+P 1450 5150
+F 0 "J10" V 1550 5150 50  0000 R CNN
+F 1 "Conn_01x04" V 1323 4862 50  0001 R CNN
+F 2 "TerminalBlock:TerminalBlock_bornier-4_P5.08mm" H 1450 5150 50  0001 C CNN
+F 3 "~" H 1450 5150 50  0001 C CNN
+	1    1450 5150
+	0    -1   -1   0
+$EndComp
 $Comp
 L Connector_Generic:Conn_01x04 J7
@@
 F 0 "J7" V 4250 3650 50  0000 R CNN
 F 1 "Conn_01x04" V 4023 3362 50  0001 R CNN
-F 2 "Connector_PinHeader_2.00mm:PinHeader_1x04_P2.00mm_Vertical" H 4150 3650 50  0001 C CNN
+F 2 "TerminalBlock:TerminalBlock_bornier-4_P5.08mm" H 4150 3650 50  0001 C CNN
 F 3 "~" H 4150 3650 50  0001 C CNN
 	1    4150 3650
 	0    -1   -1   0
 $EndComp
-$Comp
-L Connector_Generic:Conn_01x04 J9
-U 1 1 6080408C
-P 1500 3650
-F 0 "J9" V 1600 3650 50  0000 R CNN
-F 1 "Conn_01x04" V 1373 3362 50  0001 R CNN
-F 2 "Connector_PinHeader_2.00mm:PinHeader_1x04_P2.00mm_Vertical" H 1500 3650 50  0001 C CNN
-F 3 "~" H 1500 3650 50  0001 C CNN
-	1    1500 3650
-	0    -1   -1   0
-$EndComp
-$Comp
-L Connector_Generic:Conn_01x04 J10
-U 1 1 60805349
-P 1450 5150
-F 0 "J10" V 1550 5150 50  0000 R CNN
-F 1 "Conn_01x04" V 1323 4862 50  0001 R CNN
-F 2 "Connector_PinHeader_2.00mm:PinHeader_1x04_P2.00mm_Vertical" H 1450 5150 50  0001 C CNN
-F 3 "~" H 1450 5150 50  0001 C CNN
-	1    1450 5150
-	0    -1   -1   0
-$EndComp
-$Comp
-L Connector_Generic:Conn_01x04 J11
-U 1 1 608060CB
-P 2800 5150
-F 0 "J11" V 2900 5150 50  0000 R CNN
-F 1 "Conn_01x04" V 2673 4862 50  0001 R CNN
-F 2 "Connector_PinHeader_2.00mm:PinHeader_1x04_P2.00mm_Vertical" H 2800 5150 50  0001 C CNN
-F 3 "~" H 2800 5150 50  0001 C CNN
-	1    2800 5150
-	0    -1   -1   0
-$EndComp
-$Comp
-L Connector_Generic:Conn_01x04 J12
-U 1 1 60806A87
-P 4100 5150
-F 0 "J12" V 4200 5150 50  0000 R CNN
-F 1 "Conn_01x04" V 3973 4862 50  0001 R CNN
-F 2 "Connector_PinHeader_2.00mm:PinHeader_1x04_P2.00mm_Vertical" H 4100 5150 50  0001 C CNN
-F 3 "~" H 4100 5150 50  0001 C CNN
-	1    4100 5150
-	0    -1   -1   0
-$EndComp
-$Comp
-L Connector_Generic:Conn_01x04 J13
-U 1 1 608075D9
-P 5450 5150
-F 0 "J13" V 5550 5150 50  0000 R CNN
-F 1 "Conn_01x04" V 5323 4862 50  0001 R CNN
-F 2 "Connector_PinHeader_2.00mm:PinHeader_1x04_P2.00mm_Vertical" H 5450 5150 50  0001 C CNN
-F 3 "~" H 5450 5150 50  0001 C CNN
-	1    5450 5150
-	0    -1   -1   0
-$EndComp
-Wire Wire Line
-	5350 5350 5350 5450
-Wire Wire Line
-	5450 5350 5450 5400
-Wire Wire Line
-	5450 5400 5550 5400
-Wire Wire Line
-	5550 5400 5550 5450
-Wire Wire Line
-	5450 6050 5450 6200
-Wire Wire Line
-	5450 6200 5800 6200
-Wire Wire Line
-	5800 6200 5800 5450
-Wire Wire Line
-	5800 5450 5650 5450
-Wire Wire Line
-	5650 5450 5650 5350
-Wire Wire Line
-	5850 4600 5850 3950
-Wire Wire Line
-	5850 3950 5700 3950
-Wire Wire Line
-	4350 3850 4350 3950
-Wire Wire Line
-	4350 3950 4500 3950
-Wire Wire Line
-	4500 3950 4500 4600
-Wire Wire Line
-	4500 4600 4150 4600
-Wire Wire Line
-	4150 4600 4150 4550
-Wire Wire Line
-	4250 3950 4250 3900
-Wire Wire Line
-	4250 3900 4150 3900
-Wire Wire Line
-	4150 3900 4150 3850
-Wire Wire Line
-	4050 3850 4050 3950
-$Comp
-L Connector_Generic:Conn_01x04 J8
-U 1 1 60893E6F
-P 2850 3650
-F 0 "J8" V 2950 3650 50  0000 R CNN
-F 1 "Conn_01x04" V 2723 3362 50  0001 R CNN
-F 2 "Connector_PinHeader_2.00mm:PinHeader_1x04_P2.00mm_Vertical" H 2850 3650 50  0001 C CNN
-F 3 "~" H 2850 3650 50  0001 C CNN
-	1    2850 3650
-	0    -1   -1   0
-$EndComp
-Wire Wire Line
-	3050 3850 3050 3950
-Wire Wire Line
-	3050 3950 3200 3950
-Wire Wire Line
-	3200 3950 3200 4600
-Wire Wire Line
-	3200 4600 2850 4600
-Wire Wire Line
-	2850 4600 2850 4550
-Wire Wire Line
-	2850 3850 2850 3900
-Wire Wire Line
-	2850 3900 2950 3900
-Wire Wire Line
-	2950 3900 2950 3950
-Wire Wire Line
-	2750 3850 2750 3950
-Wire Wire Line
-	1400 3850 1400 3950
-Wire Wire Line
-	1500 3850 1500 3900
-Wire Wire Line
-	1500 3900 1600 3900
-Wire Wire Line
-	1600 3900 1600 3950
-Wire Wire Line
-	1700 3850 1700 4000
-Wire Wire Line
-	1700 4000 1850 4000
-Wire Wire Line
-	1850 4000 1850 4600
-Wire Wire Line
-	1850 4600 1500 4600
-Wire Wire Line
-	1500 4600 1500 4550
-Wire Wire Line
-	1350 5350 1350 5450
-Wire Wire Line
-	1450 5350 1450 5400
-Wire Wire Line
-	1450 5400 1550 5400
-Wire Wire Line
-	1550 5400 1550 5450
-Wire Wire Line
-	1650 5350 1650 5500
-Wire Wire Line
-	1650 5500 1800 5500
-Wire Wire Line
-	1800 5500 1800 6100
-Wire Wire Line
-	1800 6100 1450 6100
-Wire Wire Line
-	1450 6100 1450 6050
-Wire Wire Line
-	2700 5350 2700 5450
-Wire Wire Line
-	2800 5350 2800 5400
-Wire Wire Line
-	2800 5400 2900 5400
-Wire Wire Line
-	2900 5400 2900 5450
-Wire Wire Line
-	3000 5350 3000 5500
-Wire Wire Line
-	3000 5500 3150 5500
-Wire Wire Line
-	3150 5500 3150 6100
-Wire Wire Line
-	3150 6100 2800 6100
-Wire Wire Line
-	2800 6100 2800 6050
-Wire Wire Line
-	4000 5350 4000 5450
-Wire Wire Line
-	4100 5350 4100 5400
-Wire Wire Line
-	4100 5400 4200 5400
-Wire Wire Line
-	4200 5400 4200 5450
-Wire Wire Line
-	4300 5350 4300 5500
-Wire Wire Line
-	4300 5500 4450 5500
-Wire Wire Line
-	4450 5500 4450 6100
-Wire Wire Line
-	4450 6100 4100 6100
-Wire Wire Line
-	4100 6100 4100 6050
+Wire Wire Line
+	7250 4350 7350 4350
 $EndSCHEMATC

Commit message: att
Connections:
- net +12V: no longer U2.10 (~SRCLR)
- net +5V: now also U2.10 (~SRCLR)
Changed lines of the file:
@@
 	1    0    0    -1
 $EndComp
-$Comp
-L power:+12V #PWR0115
-U 1 1 606A4273
-P 3850 1800
-F 0 "#PWR0115" H 3850 1650 50  0001 C CNN
-F 1 "+12V" H 3865 1973 50  0000 C CNN
-F 2 "" H 3850 1800 50  0001 C CNN
-F 3 "" H 3850 1800 50  0001 C CNN
-	1    3850 1800
-	-1   0    0    1
-$EndComp
 Wire Wire Line
 	4150 1600 4050 1600
 Wire Wire Line
 	4050 1600 4050 1800
-Wire Wire Line
-	3850 1300 3850 1800
 Wire Wire Line
 	3850 1300 4150 1300
@@
 Wire Wire Line
 	7250 4350 7350 4350
+Text HLabel 3850 1850 3    50   Input ~ 0
++5V
+Wire Wire Line
+	3850 1850 3850 1300
 $EndSCHEMATC
