File: kicad_Poolcontroller/kicad_Poolcontroller.kicad_pcb (KiCad board)
At the start: 2 copper layers, 47 parts, among them J1 Conn_02x01, J2 Conn_02x02_Odd_Even, J3 Conn_02x02_Odd_Even, J4 Conn_02x01, K1 SANYOU_SRD_Form_C, K2 SANYOU_SRD_Form_C, K3 SANYOU_SRD_Form_C, K4 SANYOU_SRD_Form_C, K5 SANYOU_SRD_Form_C, K6 SANYOU_SRD_Form_C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

Commit message: att
Parts:
- added J10: Conn_02x01, TerminalBlock:TerminalBlock_bornier-2_P5.08mm, F.Cu at (169.0, 93.5)
- added J11: Conn_02x01, TerminalBlock:TerminalBlock_bornier-2_P5.08mm, F.Cu at (169.0, 73.5)
- added J12: Conn_02x01, TerminalBlock:TerminalBlock_bornier-2_P5.08mm, F.Cu at (169.0, 53.5)
- added J13: Conn_02x01, TerminalBlock:TerminalBlock_bornier-2_P5.08mm, F.Cu at (169.0, 33.5)
- added J5: ESP01, Connector_PinSocket_2.54mm:PinSocket_2x04_P2.54mm_Vertical, F.Cu at (79.0, 75.0)
- added J6: Conn_01x03, TerminalBlock:TerminalBlock_bornier-3_P5.08mm, F.Cu at (20.0, 101.1)
- added J7: Conn_02x01, TerminalBlock:TerminalBlock_bornier-2_P5.08mm, F.Cu at (20.0, 78.5)
- added J8: Conn_02x01, TerminalBlock:TerminalBlock_bornier-2_P5.08mm, F.Cu at (20.0, 58.5)
- added J9: Conn_02x01, TerminalBlock:TerminalBlock_bornier-2_P5.08mm, F.Cu at (20.0, 38.5)
- C1, C2, C3, C4: footprint Capacitor_THT:CP_Radial_D8.0mm_P3.50mm -> Capacitor_THT:CP_Radial_D5.0mm_P2.50mm
- J4: value Conn_02x01 -> Conn_01x04; footprint Connector_PinHeader_2.54mm:PinHeader_2x01_P2.54mm_Vertical -> Connector_PinSocket_2.54mm:PinSocket_1x04_P2.54mm_Vertical
- Q1, Q2, Q3, Q4, Q5, Q6, Q7, Q8: footprint Package_TO_SOT_THT:TO-39-3 -> Package_TO_SOT_THT:TO-92
- U1: footprint Package_DIP:DIP-6_W7.62mm_Socket -> Package_DIP:DIP-8_W7.62mm_Socket
- U5: footprint Package_TO_SOT_THT:TO-220-3_Vertical -> Package_TO_SOT_THT:TO-220-3_Horizontal_TabDown
- moved Q3 151.3 mm to (57.0, 74.5), turned to 270 degrees
- moved C1 145.0 mm to (70.0, 39.0)
- moved Q1 142.4 mm to (57.0, 34.5), turned to 270 degrees
- moved Q4 130.8 mm to (57.0, 94.5), turned to 270 degrees
- moved D8 130.2 mm to (138.0, 31.0), turned to 270 degrees
- moved K8 129.8 mm to (145.0, 36.0)
- moved J1 126.3 mm to (65.0, 30.0)
- moved Q2 123.6 mm to (57.0, 54.5), turned to 270 degrees
- moved C2 117.2 mm to (79.5, 39.0)
- moved J2 114.4 mm to (74.0, 30.0)
- moved C3 104.8 mm to (107.0, 39.0)
- moved U1 103.9 mm to (92.0, 40.0)
- moved K1 103.4 mm to (44.0, 36.0), turned to 180 degrees
- moved C4 102.4 mm to (116.0, 39.0)
- moved U3 102.2 mm to (87.0, 31.5)
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Connections:
- J3 pad 2: Net-(J3-Pad2) -> +12V
- J3 pad 3: Net-(J3-Pad3) -> GND
- J4 pad 1: Net-(J4-Pad1) -> /+3.3V
- J4 pad 2: +12V -> /TX
- K1 pad 1: Net-(J4-Pad1) -> Net-(K1-Pad1)
- K2 pad 1: Net-(J4-Pad1) -> Net-(K2-Pad1)
- K3 pad 1: Net-(J4-Pad1) -> Net-(K3-Pad1)
- K4 pad 1: Net-(J4-Pad1) -> Net-(J6-Pad2)
- K5 pad 1: Net-(J4-Pad1) -> Net-(K5-Pad1)
- K6 pad 1: Net-(J4-Pad1) -> Net-(K6-Pad1)
- K7 pad 1: Net-(J4-Pad1) -> Net-(K7-Pad1)
- K8 pad 1: Net-(J4-Pad1) -> Net-(K8-Pad1)
- Q1 pad 3: +12V -> Net-(J3-Pad1)
- Q2 pad 3: +12V -> Net-(J3-Pad1)
- Q3 pad 3: +12V -> Net-(J3-Pad1)
- Q4 pad 3: +12V -> Net-(J3-Pad1)
- Q5 pad 3: +12V -> Net-(J3-Pad1)
- Q6 pad 3: +12V -> Net-(J3-Pad1)
- Q7 pad 3: +12V -> Net-(J3-Pad1)
- Q8 pad 3: +12V -> Net-(J3-Pad1)
- U1 pad 1: Net-(U1-Pad1) -> /EN
- U1 pad 2: Net-(J3-Pad4) -> /RX
- U1 pad 3: Net-(J3-Pad2) -> /TX
- U2 pad 10: Net-(U1-Pad6) -> +12V
- U2 pad 13: Net-(U2-Pad13) -> GND
- U2 pad 14: Net-(U2-Pad14) -> Net-(U1-Pad6)
Routing:
- net Net-(J9-Pad2): track 0.00 -> 11.3 mm
- net Net-(J8-Pad2): track 0.00 -> 11.3 mm
- net Net-(J7-Pad2): track 0.00 -> 11.3 mm
- net Net-(J9-Pad1): track 0.00 -> 11.2 mm
- net Net-(J7-Pad1): track 0.00 -> 11.2 mm
Other:
- board text added: "+12V"
- board text added: "+5V"
- board text added: "74HC595"
- board text added: "7805"
- board text added: "7809"
- board text added: "ATtiny85"
- board text added: "Alim"
- board text added: "Alim."
- board text added: "GND"
- board text added: "J4"
- board text added: "J5"
- board text added: "Jumper"
- board text added: "LM317"

Commit message: att
Parts:
- J10, J11, J12, J13, J7, J8, J9: value Conn_02x01 -> Conn_01x04; footprint TerminalBlock:TerminalBlock_bornier-2_P5.08mm -> Connector_PinHeader_2.00mm:PinHeader_1x04_P2.00mm_Vertical
- J6: value Conn_01x03 -> Conn_01x04; footprint TerminalBlock:TerminalBlock_bornier-3_P5.08mm -> Connector_PinHeader_2.00mm:PinHeader_1x04_P2.00mm_Vertical
- moved J10 170.6 mm to (4.77, 47.5), turned to 0 degrees
- moved J11 162.3 mm to (8.82, 47.5), turned to 0 degrees
- moved J12 156.2 mm to (12.9, 47.5), turned to 0 degrees
- moved J13 152.7 mm to (16.9, 47.5), turned to 0 degrees
- moved J6 62.1 mm to (-11.4, 47.5), turned to 0 degrees
- moved J7 41.4 mm to (-7.38, 47.5), turned to 0 degrees
- moved J8 25.8 mm to (-3.33, 47.5), turned to 0 degrees
- moved J9 21.3 mm to (0.72, 47.5), turned to 0 degrees
Connections:
- K1 pad 1: Net-(K1-Pad1) -> Net-(J9-Pad4)
- K2 pad 1: Net-(K2-Pad1) -> Net-(J8-Pad4)
- K3 pad 1: Net-(K3-Pad1) -> Net-(J7-Pad4)
- K4 pad 1: Net-(J6-Pad2) -> Net-(J6-Pad4)
- K4 pad 3: Net-(J6-Pad3) -> Net-(J6-Pad2)
- K5 pad 1: Net-(K5-Pad1) -> Net-(J10-Pad4)
- K6 pad 1: Net-(K6-Pad1) -> Net-(J11-Pad4)
- K7 pad 1: Net-(K7-Pad1) -> Net-(J12-Pad4)
- K8 pad 1: Net-(K8-Pad1) -> Net-(J13-Pad4)

Commit message: att
Parts:
- J10, J11, J12, J13, J6, J7, J8, J9: footprint Connector_PinHeader_2.00mm:PinHeader_1x04_P2.00mm_Vertical -> TerminalBlock:TerminalBlock_bornier-4_P5.08mm
- moved J10 171.1 mm to (170.0, 92.0), turned to 270 degrees
- moved J11 162.9 mm to (170.0, 71.0), turned to 270 degrees
- moved J12 157.1 mm to (170.0, 50.0), turned to 270 degrees
- moved J13 154.2 mm to (170.0, 29.0), turned to 270 degrees
- moved J6 67.3 mm to (20.0, 107.0), turned to 90 degrees
- moved J7 47.2 mm to (20.0, 86.0), turned to 90 degrees
- moved J8 29.2 mm to (20.0, 65.0), turned to 90 degrees
- moved J9 19.6 mm to (20.0, 44.0), turned to 90 degrees
- moved D4 3.00 mm to (51.0, 104.0)
- moved D5 3.00 mm to (138.0, 94.0)
- moved K4 3.00 mm to (44.0, 99.0)
- moved K5 3.00 mm to (145.0, 99.0)
- moved Q4 3.00 mm to (57.0, 97.5)
- moved D3 2.00 mm to (51.0, 83.0)
- moved D6 2.00 mm to (138.0, 73.0)
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Routing:
- net Net-(J9-Pad2): track 11.3 -> 0.00 mm
- net Net-(J8-Pad2): track 11.3 -> 0.00 mm
- net Net-(J7-Pad2): track 11.3 -> 0.00 mm
- net Net-(J9-Pad1): track 11.2 -> 0.00 mm
- net Net-(J7-Pad1): track 11.2 -> 0.00 mm
Other:
- board text added: "COM"
- board text added: "NC"
- board text added: "NF"
- board text added: "NO"

Commit message: att
Parts:
- ESP - 01: renamed from J5
- moved J10 1.00 mm to (170.0, 91.0)
- moved J11 1.00 mm to (170.0, 70.0)
- moved J12 1.00 mm to (170.0, 49.0)
- moved J13 1.00 mm to (170.0, 28.0)
- renumbered J4 to 433MHz
Routing:
- net Net-(J12-Pad4): track 0.00 -> 29.2 mm
- net Net-(J11-Pad4): track 0.00 -> 29.2 mm
- net Net-(J10-Pad4): track 0.00 -> 29.2 mm
- net Net-(J13-Pad4): track 0.00 -> 29.2 mm
- net Net-(J7-Pad4): track 0.00 -> 28.3 mm
- net Net-(J6-Pad4): track 0.00 -> 28.3 mm
- net Net-(J9-Pad4): track 0.00 -> 28.3 mm
- net Net-(J8-Pad4): track 0.00 -> 28.3 mm
- net Net-(J13-Pad2): track 0.00 -> 17.1 mm
- net Net-(J12-Pad2): track 0.00 -> 17.1 mm
- net Net-(J11-Pad2): track 0.00 -> 17.1 mm
- net Net-(J10-Pad2): track 0.00 -> 17.1 mm
- net Net-(J9-Pad2): track 0.00 -> 15.9 mm
- net Net-(J8-Pad2): track 0.00 -> 15.9 mm
- net Net-(J7-Pad2): track 0.00 -> 15.9 mm
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Changed lines of the file:
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@@
     (thickness 1.6)
     (drawings 47)
-    (tracks 0)
+    (tracks 80)
     (zones 0)
     (modules 56)
@@
   )
   (setup
-    (last_trace_width 0.25)
+    (last_trace_width 1.8)
     (user_trace_width 0.2)
     (user_trace_width 0.4)
@@
   )
   (module TerminalBlock:TerminalBlock_bornier-4_P5.08mm (layer F.Cu)
-    (at 170 29 270)
+    (at 170 28 270)
     (descr "simple 4-pin terminal block, pitch 5.08mm, revamped version of bornier4")
     (tags "terminal block bornier4")
@@
   )
   (module TerminalBlock:TerminalBlock_bornier-4_P5.08mm (layer F.Cu)
-    (at 170 50 270)
+    (at 170 49 270)
     (descr "simple 4-pin terminal block, pitch 5.08mm, revamped version of bornier4")
     (tags "terminal block bornier4")
@@
   )
   (module TerminalBlock:TerminalBlock_bornier-4_P5.08mm (layer F.Cu)
-    (at 170 71 270)
+    (at 170 70 270)
     (descr "simple 4-pin terminal block, pitch 5.08mm, revamped version of bornier4")
     (tags "terminal block bornier4")
@@
   )
   (module TerminalBlock:TerminalBlock_bornier-4_P5.08mm (layer F.Cu)
-    (at 170 92 270)
+    (at 170 91 270)
     (descr "simple 4-pin terminal block, pitch 5.08mm, revamped version of bornier4")
     (tags "terminal block bornier4")
@@
     (descr "Through hole straight socket strip, 2x04, 2.54mm pitch, double cols (from Kicad 4.0.7), script generated")
     (tags "Through hole socket strip THT 2x04 2.54mm double row")
-    (fp_text reference J5 (at 3 4 180) (layer F.SilkS)
+    (fp_text reference "ESP - 01" (at 3 4 180) (layer F.SilkS)
       (effects (font (size 1 1) (thickness 0.15)))
     )
@@
     (descr "Through hole straight socket strip, 1x04, 2.54mm pitch, single row (from Kicad 4.0.7), script generated")
     (tags "Through hole socket strip THT 1x04 2.54mm single row")
-    (fp_text reference J4 (at -3 4 180) (layer F.SilkS)
+    (fp_text reference 433MHz (at -3 4 180) (layer F.SilkS)
       (effects (font (size 1 1) (thickness 0.15)))
     )
@@
     (effects (font (size 1 1) (thickness 0.15)))
   )
-  (gr_text "J4\n" (at 106.172 72.136) (layer F.SilkS)
+  (gr_text "J4\n" (at 106.172 71.882) (layer F.SilkS)
     (effects (font (size 1 1) (thickness 0.15)))
   )
-  (gr_text J5 (at 84.074 73.152) (layer F.SilkS)
+  (gr_text J5 (at 82.296 73.152) (layer F.SilkS)
     (effects (font (size 1 1) (thickness 0.15)))
   )
@@
     (arrow2b (pts (xy 45.288 45.728) (xy 45.874421 46.854504)))
   )
+  (segment (start 29.85 92.95) (end 29.85 96.904) (width 1.8) (layer B.Cu) (net 47))
+  (segment (start 24.834 38.92) (end 20 38.92) (width 1.8) (layer B.Cu) (net 53))
+  (segment (start 29.85 29.95) (end 29.85 33.904) (width 1.8) (layer B.Cu) (net 53))
+  (segment (start 29.85 71.95) (end 29.85 75.904) (width 1.8) (layer B.Cu) (net 49))
+  (segment (start 29.85 33.904) (end 24.834 38.92) (width 1.8) (layer B.Cu) (net 53))
+  (segment (start 29.85 54.904) (end 24.834 59.92) (width 1.8) (layer B.Cu) (net 51))
+  (segment (start 29.85 75.904) (end 24.834 80.92) (width 1.8) (layer B.Cu) (net 49))
+  (segment (start 29.85 96.904) (end 24.834 101.92) (width 1.8) (layer B.Cu) (net 47))
+  (segment (start 24.834 59.92) (end 20 59.92) (width 1.8) (layer B.Cu) (net 51))
+  (segment (start 24.834 80.92) (end 20 80.92) (width 1.8) (layer B.Cu) (net 49))
+  (segment (start 24.834 101.92) (end 20 101.92) (width 1.8) (layer B.Cu) (net 47))
+  (segment (start 20 44) (end 27.8 44) (width 1.8) (layer B.Cu) (net 54))
+  (segment (start 20 107) (end 27.8 107) (width 1.8) (layer B.Cu) (net 48))
+  (segment (start 27.8 86) (end 29.8 84) (width 1.8) (layer B.Cu) (net 50))
+  (segment (start 27.8 107) (end 29.8 105) (width 1.8) (layer B.Cu) (net 48))
+  (segment (start 20 86) (end 27.8 86) (width 1.8) (layer B.Cu) (net 50))
+  (segment (start 29.85 50.95) (end 29.85 54.904) (width 1.8) (layer B.Cu) (net 51))
+  (segment (start 27.8 65) (end 29.8 63) (width 1.8) (layer B.Cu) (net 52))
+  (segment (start 20 65) (end 27.8 65) (width 1.8) (layer B.Cu) (net 52))
+  (segment (start 27.8 44) (end 29.8 42) (width 1.8) (layer B.Cu) (net 54))
+  (segment (start 159.15 42.05) (end 159.15 37.7) (width 1.8) (layer B.Cu) (net 61))
+  (segment (start 163.77 33.08) (end 170 33.08) (width 1.8) (layer B.Cu) (net 61))
+  (segment (start 159.15 37.7) (end 163.77 33.08) (width 1.8) (layer B.Cu) (net 61))
+  (segment (start 161.2 28) (end 159.2 30) (width 1.8) (layer B.Cu) (net 62))
+  (segment (start 170 28) (end 161.2 28) (width 1.8) (layer B.Cu) (net 62))
+  (segment (start 170 49) (end 161.2 49) (width 1.8) (layer B.Cu) (net 60))
+  (segment (start 170 70) (end 161.2 70) (width 1.8) (layer B.Cu) (net 58))
+  (segment (start 170 91) (end 161.2 91) (width 1.8) (layer B.Cu) (net 56))
+  (segment (start 161.2 49) (end 159.2 51) (width 1.8) (layer B.Cu) (net 60))
+  (segment (start 161.2 70) (end 159.2 72) (width 1.8) (layer B.Cu) (net 58))
+  (segment (start 161.2 91) (end 159.2 93) (width 1.8) (layer B.Cu) (net 56))
+  (segment (start 163.77 54.08) (end 170 54.08) (width 1.8) (layer B.Cu) (net 59))
+  (segment (start 163.77 75.08) (end 170 75.08) (width 1.8) (layer B.Cu) (net 57))
+  (segment (start 163.77 96.08) (end 170 96.08) (width 1.8) (layer B.Cu) (net 55))
+  (segment (start 159.15 58.7) (end 163.77 54.08) (width 1.8) (layer B.Cu) (net 59))
+  (segment (start 159.15 79.7) (end 163.77 75.08) (width 1.8) (layer B.Cu) (net 57))
+  (segment (start 159.15 100.7) (end 163.77 96.08) (width 1.8) (layer B.Cu) (net 55))
+  (segment (start 159.15 63.05) (end 159.15 58.7) (width 1.8) (layer B.Cu) (net 59))
+  (segment (start 159.15 84.05) (end 159.15 79.7) (width 1.8) (layer B.Cu) (net 57))
+  (segment (start 159.15 105.05) (end 159.15 100.7) (width 1.8) (layer B.Cu) (net 55))
+  (segment (start 24.326 28.76) (end 25.908 27.178) (width 1.8) (layer B.Cu) (net 69))
+  (segment (start 39.748002 36) (end 44 36) (width 1.8) (layer B.Cu) (net 69))
+  (segment (start 30.926002 27.178) (end 39.748002 36) (width 1.8) (layer B.Cu) (net 69))
+  (segment (start 25.908 27.178) (end 30.926002 27.178) (width 1.8) (layer B.Cu) (net 69))
+  (segment (start 39.748002 57) (end 44 57) (width 1.8) (layer B.Cu) (net 67))
+  (segment (start 39.748002 78) (end 44 78) (width 1.8) (layer B.Cu) (net 65))
+  (segment (start 39.748002 99) (end 44 99) (width 1.8) (layer B.Cu) (net 64))
+  (segment (start 30.926002 48.178) (end 39.748002 57) (width 1.8) (layer B.Cu) (net 67))
+  (segment (start 30.926002 69.178) (end 39.748002 78) (width 1.8) (layer B.Cu) (net 65))
+  (segment (start 30.926002 90.178) (end 39.748002 99) (width 1.8) (layer B.Cu) (net 64))
+  (segment (start 25.908 48.178) (end 30.926002 48.178) (width 1.8) (layer B.Cu) (net 67))
+  (segment (start 25.908 69.178) (end 30.926002 69.178) (width 1.8) (layer B.Cu) (net 65))
+  (segment (start 25.908 90.178) (end 30.926002 90.178) (width 1.8) (layer B.Cu) (net 64))
+  (segment (start 20 28.76) (end 24.326 28.76) (width 1.8) (layer B.Cu) (net 69))
+  (segment (start 24.326 49.76) (end 25.908 48.178) (width 1.8) (layer B.Cu) (net 67))
+  (segment (start 24.326 70.76) (end 25.908 69.178) (width 1.8) (layer B.Cu) (net 65))
+  (segment (start 24.326 91.76) (end 25.908 90.178) (width 1.8) (layer B.Cu) (net 64))
+  (segment (start 20 49.76) (end 24.326 49.76) (width 1.8) (layer B.Cu) (net 67))
+  (segment (start 20 70.76) (end 24.326 70.76) (width 1.8) (layer B.Cu) (net 65))
+  (segment (start 20 91.76) (end 24.326 91.76) (width 1.8) (layer B.Cu) (net 64))
+  (segment (start 149.251998 36) (end 145 36) (width 1.8) (layer B.Cu) (net 77))
+  (segment (start 157.901999 44.650001) (end 149.251998 36) (width 1.8) (layer B.Cu) (net 77))
+  (segment (start 163.749999 44.650001) (end 157.901999 44.650001) (width 1.8) (layer B.Cu) (net 77))
+  (segment (start 165.16 43.24) (end 163.749999 44.650001) (width 1.8) (layer B.Cu) (net 77))
+  (segment (start 170 43.24) (end 165.16 43.24) (width 1.8) (layer B.Cu) (net 77))
+  (segment (start 170 64.24) (end 165.16 64.24) (width 1.8) (layer B.Cu) (net 75))
+  (segment (start 170 85.24) (end 165.16 85.24) (width 1.8) (layer B.Cu) (net 73))
+  (segment (start 170 106.24) (end 165.16 106.24) (width 1.8) (layer B.Cu) (net 71))
+  (segment (start 165.16 64.24) (end 163.749999 65.650001) (width 1.8) (layer B.Cu) (net 75))
+  (segment (start 165.16 85.24) (end 163.749999 86.650001) (width 1.8) (layer B.Cu) (net 73))
+  (segment (start 165.16 106.24) (end 163.749999 107.650001) (width 1.8) (layer B.Cu) (net 71))
+  (segment (start 163.749999 65.650001) (end 157.901999 65.650001) (width 1.8) (layer B.Cu) (net 75))
+  (segment (start 163.749999 86.650001) (end 157.901999 86.650001) (width 1.8) (layer B.Cu) (net 73))
+  (segment (start 163.749999 107.650001) (end 157.901999 107.650001) (width 1.8) (layer B.Cu) (net 71))
+  (segment (start 157.901999 65.650001) (end 149.251998 57) (width 1.8) (layer B.Cu) (net 75))
+  (segment (start 157.901999 86.650001) (end 149.251998 78) (width 1.8) (layer B.Cu) (net 73))
+  (segment (start 157.901999 107.650001) (end 149.251998 99) (width 1.8) (layer B.Cu) (net 71))
+  (segment (start 149.251998 57) (end 145 57) (width 1.8) (layer B.Cu) (net 75))
+  (segment (start 149.251998 78) (end 145 78) (width 1.8) (layer B.Cu) (net 73))
+  (segment (start 149.251998 99) (end 145 99) (width 1.8) (layer B.Cu) (net 71))
 )

Commit message: att
Parts:
- J5: renamed from ESP - 01
- moved Q1 2.97 mm to (58.0, 37.3), turned to 90 degrees
- moved Q2 2.97 mm to (58.0, 58.3), turned to 90 degrees
- moved Q3 2.97 mm to (58.0, 79.3), turned to 90 degrees
- moved Q4 2.97 mm to (58.0, 100.3), turned to 90 degrees
- moved Q8 2.97 mm to (131.0, 34.7), turned to 270 degrees
- moved Q7 1.56 mm to (131.0, 56.3), turned to 270 degrees
- moved Q6 1.28 mm to (131.0, 76.7), turned to 270 degrees
- moved Q5 1.02 mm to (131.0, 97.7), turned to 270 degrees
- moved J3 0.25 mm to (122.7, 30.0)
- renumbered 433MHz to J4
Connections:
- J2 pad 4: Net-(J2-Pad4) -> /+5V
Routing:
- net GND: track 0.00 -> 272.4 mm
- net /Q4: track 0.00 -> 41.3 mm
- net /Q3: track 0.00 -> 26.8 mm
- net /Q1: track 0.00 -> 19.5 mm
- net /K6: track 0.00 -> 19.1 mm
- net /K5: track 0.00 -> 19.1 mm
- net /K8: track 0.00 -> 19.1 mm
- net /K7: track 0.00 -> 19.1 mm
- net /Q5: track 0.00 -> 19.1 mm
- net /K4: track 0.00 -> 19.0 mm
- net /K3: track 0.00 -> 19.0 mm
- net /K2: track 0.00 -> 19.0 mm
- net /K1: track 0.00 -> 19.0 mm
- net /Q8: track 0.00 -> 18.2 mm
- net /Q2: track 0.00 -> 16.1 mm
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
Commit message: att
Parts:
- moved U1 11.0 mm to (99.5, 48.0), turned to 180 degrees
- moved C2 2.50 mm to (82.0, 39.0), turned to 180 degrees
Connections:
- U2 pad 10: +12V -> /+5V
Routing:
- net GND: track 272.4 -> 637.4 mm
- net Net-(J3-Pad1): track 0.00 -> 295.8 mm, vias 0 -> 6
- net /+3.3V: track 0.00 -> 84.6 mm
- net Net-(C4-Pad1): track 0.00 -> 82.6 mm, vias 0 -> 8
- net /TX: track 0.00 -> 69.6 mm
- net +12V: track 14.3 -> 78.4 mm, vias 0 -> 4
- net /EN: track 0.00 -> 59.4 mm, vias 0 -> 4
- net /+5V: track 0.00 -> 52.5 mm, vias 0 -> 6
- net Net-(C2-Pad1): track 0.00 -> 38.6 mm
- net Net-(R2-Pad1): track 0.00 -> 35.1 mm
- net /RX: track 0.00 -> 34.4 mm
- net Net-(R1-Pad1): track 0.00 -> 30.4 mm
- net Net-(R4-Pad1): track 0.00 -> 30.0 mm
- net Net-(C1-Pad1): track 11.1 -> 40.9 mm
- net Net-(R7-Pad1): track 0.00 -> 24.5 mm
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
Commit message: att
Parts:
- moved J3 56.4 mm to (176.3, 47.5)
- moved C1 56.4 mm to (123.6, 56.5)
- moved C2 56.4 mm to (135.6, 56.5)
- moved C3 56.4 mm to (160.6, 56.5)
- moved C4 56.4 mm to (169.6, 56.5)
- moved D1 56.4 mm to (104.6, 58.5)
- moved D2 56.4 mm to (104.6, 79.5)
- moved D3 56.4 mm to (104.6, 100.5)
- moved D4 56.4 mm to (104.6, 121.5)
- moved D5 56.4 mm to (191.6, 111.5)
- moved D6 56.4 mm to (191.6, 90.5)
- moved D7 56.4 mm to (191.6, 69.5)
- moved D8 56.4 mm to (191.6, 48.5)
- moved J1 56.4 mm to (118.6, 47.5)
- moved J10 56.4 mm to (223.6, 108.5)
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Routing:
- net /RX: track 34.4 -> 117.4 mm, vias 0 -> 4
- net /+5V: track 52.5 -> 63.0 mm, vias 6 -> 7
- net +12V: track 78.4 -> 74.8 mm
- net (no net): vias 0 -> 4
- added copper zone on B.Cu, net (none)
