File: kicad_Servo/kicad_Poolcontroller.sch (KiCad schematic (older format))
At the start: 52 parts, among them J1 Conn_02x02_Odd_Even, J10 Conn_01x04, J11 Conn_01x04, J12 Conn_01x04, J13 Conn_01x04, J4 Conn_01x04, J5 ESP01, J6 Conn_01x04, J7 Conn_01x04, J8 Conn_01x04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

Commit message: .
Parts:
- J4: value Conn_01x04 -> RF
Changed lines of the file:
@@
 encoding utf-8
 Sheet 1 1
-Title ""
-Date ""
+Title "pcb_servoAttiny"
+Date "2021-05-19"
 Rev ""
 Comp ""
@@
 U 1 1 607CD9BA
 P 2350 4000
-F 0 "J4" H 2268 3575 50  0000 C CNN
-F 1 "Conn_01x04" H 2268 3666 50  0000 C CNN
+F 0 "J4" H 2350 3600 50  0000 C CNN
+F 1 "RF " H 2329 3700 50  0000 C CNN
 F 2 "Connector_PinSocket_2.54mm:PinSocket_1x04_P2.54mm_Vertical" H 2350 4000 50  0001 C CNN
 F 3 "~" H 2350 4000 50  0001 C CNN
